File: baikal_be-t100.kicad_pcb (KiCad board)
At the start: 2 copper layers, 0 parts

Commit message: Work in progress...
Parts:
- added DD1: Baikal_BE-T1000, Housing_BGA_Baikal:BGA-576_24x24_25.0x25.0mm, F.Cu at (-48.9, -47.8)
- added J1: 2-2013289-1, 2-2013289-1:TE_2-2013289-1, B.Cu at (-70.1, -45.7)
Other:
- board outline added: 95.9 x 90.2 mm

Commit message: Work in progress...
Connections:
- DD1 pad A1: (no net) -> Net-(DD1-PadA1)
- DD1 pad A15: (no net) -> Net-(DD1-PadA1)
- DD1 pad A22: (no net) -> Net-(DD1-PadA1)
- DD1 pad A23: (no net) -> GNDD
- DD1 pad A8: (no net) -> Net-(DD1-PadA1)
- DD1 pad AA3: (no net) -> GNDD
- DD1 pad AB12: (no net) -> GNDD
- DD1 pad AB14: (no net) -> GNDD
- DD1 pad AB15: (no net) -> GNDD
- DD1 pad AB17: (no net) -> GNDD
- DD1 pad AB19: (no net) -> GNDD
- DD1 pad AB20: (no net) -> GNDD
- DD1 pad AB21: (no net) -> GNDD
- DD1 pad AB4: (no net) -> Net-(DD1-PadA1)
- DD1 pad AB5: (no net) -> GNDD
- DD1 pad AB7: (no net) -> GNDD
- DD1 pad AB9: (no net) -> GNDD
- DD1 pad AC1: (no net) -> Net-(DD1-PadA1)
- DD1 pad AC19: (no net) -> Net-(DD1-PadA1)
- DD1 pad AC20: (no net) -> Net-(DD1-PadA1)
- DD1 pad AD2: (no net) -> GNDD
- DD1 pad AD23: (no net) -> GNDD
- DD1 pad B1: (no net) -> GNDD
- DD1 pad B15: (no net) -> GNDD
- DD1 pad B8: (no net) -> GNDD
- DD1 pad C16: (no net) -> GNDD
- DD1 pad C21: (no net) -> GNDD
- DD1 pad E1: (no net) -> Net-(DD1-PadA1)
- DD1 pad E16: (no net) -> Net-(DD1-PadA1)
- DD1 pad E17: (no net) -> GNDD
- DD1 pad E19: (no net) -> GNDD
- DD1 pad E2: (no net) -> GNDD
- DD1 pad F18: (no net) -> GNDD
- DD1 pad G10: (no net) -> Net-(DD1-PadA1)
- DD1 pad G11: (no net) -> Net-(DD1-PadA1)
- DD1 pad G12: (no net) -> Net-(DD1-PadA1)
- DD1 pad G13: (no net) -> Net-(DD1-PadA1)
- DD1 pad G14: (no net) -> Net-(DD1-PadA1)
- DD1 pad G15: (no net) -> Net-(DD1-PadA1)
- DD1 pad G16: (no net) -> Net-(DD1-PadA1)
- DD1 pad G22: (no net) -> Net-(DD1-PadA1)
- DD1 pad G23: (no net) -> GNDD
- DD1 pad G8: (no net) -> Net-(DD1-PadA1)
- DD1 pad G9: (no net) -> Net-(DD1-PadA1)
- DD1 pad H10: (no net) -> GNDD
- DD1 pad H11: (no net) -> GNDD
- DD1 pad H12: (no net) -> GNDD
- DD1 pad H13: (no net) -> GNDD
- DD1 pad H14: (no net) -> GNDD
- DD1 pad H15: (no net) -> GNDD
- DD1 pad H16: (no net) -> GNDD
- DD1 pad H18: (no net) -> GNDD
- DD1 pad H8: (no net) -> GNDD
- DD1 pad H9: (no net) -> GNDD
- DD1 pad J10: (no net) -> Net-(DD1-PadA1)
- DD1 pad J11: (no net) -> Net-(DD1-PadA1)
- DD1 pad J12: (no net) -> Net-(DD1-PadA1)
- DD1 pad J13: (no net) -> Net-(DD1-PadA1)
- DD1 pad J14: (no net) -> Net-(DD1-PadA1)
- DD1 pad J15: (no net) -> Net-(DD1-PadA1)
- DD1 pad J16: (no net) -> Net-(DD1-PadA1)
- DD1 pad J23: (no net) -> GNDD
- DD1 pad J8: (no net) -> Net-(DD1-PadA1)
- DD1 pad J9: (no net) -> Net-(DD1-PadA1)
- DD1 pad K10: (no net) -> GNDD
- DD1 pad K11: (no net) -> GNDD
- DD1 pad K12: (no net) -> GNDD
- DD1 pad K13: (no net) -> GNDD
- DD1 pad K14: (no net) -> GNDD
- DD1 pad K15: (no net) -> GNDD
- DD1 pad K16: (no net) -> GNDD
- DD1 pad K20: (no net) -> GNDD
- DD1 pad K8: (no net) -> GNDD
- DD1 pad K9: (no net) -> GNDD
- DD1 pad L10: (no net) -> Net-(DD1-PadA1)
- DD1 pad L11: (no net) -> Net-(DD1-PadA1)
- DD1 pad L12: (no net) -> Net-(DD1-PadA1)
- DD1 pad L13: (no net) -> Net-(DD1-PadA1)
- DD1 pad L14: (no net) -> Net-(DD1-PadA1)
- DD1 pad L15: (no net) -> Net-(DD1-PadA1)
- DD1 pad L16: (no net) -> Net-(DD1-PadL16)
- DD1 pad L18: (no net) -> GNDD
- DD1 pad L23: (no net) -> GNDD
- DD1 pad L8: (no net) -> Net-(DD1-PadL16)
- DD1 pad L9: (no net) -> Net-(DD1-PadL16)
- DD1 pad M1: (no net) -> Net-(DD1-PadL16)
- DD1 pad M10: (no net) -> GNDD
- DD1 pad M11: (no net) -> GNDD
- DD1 pad M12: (no net) -> GNDD
- DD1 pad M13: (no net) -> GNDD
- DD1 pad M14: (no net) -> GNDD
- DD1 pad M15: (no net) -> GNDD
- DD1 pad M16: (no net) -> GNDD
- DD1 pad M2: (no net) -> GNDD
- DD1 pad M8: (no net) -> GNDD
- DD1 pad M9: (no net) -> GNDD
- DD1 pad N10: (no net) -> Net-(DD1-PadL16)
- DD1 pad N11: (no net) -> Net-(DD1-PadL16)
- DD1 pad N12: (no net) -> Net-(DD1-PadL16)
- DD1 pad N13: (no net) -> Net-(DD1-PadL16)
- DD1 pad N14: (no net) -> Net-(DD1-PadL16)
- DD1 pad N15: (no net) -> Net-(DD1-PadL16)
- DD1 pad N16: (no net) -> Net-(DD1-PadL16)
- DD1 pad N17: (no net) -> GNDD
- DD1 pad N20: (no net) -> GNDD
- DD1 pad N23: (no net) -> GNDD
- DD1 pad N8: (no net) -> Net-(DD1-PadL16)
- DD1 pad N9: (no net) -> Net-(DD1-PadL16)
- DD1 pad P10: (no net) -> GNDD
- DD1 pad P11: (no net) -> GNDD
- DD1 pad P12: (no net) -> GNDD
- DD1 pad P13: (no net) -> GNDD
- DD1 pad P14: (no net) -> GNDD
- DD1 pad P15: (no net) -> GNDD
- DD1 pad P16: (no net) -> GNDD
- DD1 pad P8: (no net) -> GNDD
- DD1 pad P9: (no net) -> GNDD
- DD1 pad R10: (no net) -> Net-(DD1-PadL16)
- DD1 pad R11: (no net) -> Net-(DD1-PadL16)
- DD1 pad R12: (no net) -> Net-(DD1-PadL16)
- DD1 pad R13: (no net) -> Net-(DD1-PadL16)
- DD1 pad R14: (no net) -> Net-(DD1-PadL16)
- DD1 pad R15: (no net) -> Net-(DD1-PadL16)
- DD1 pad R16: (no net) -> Net-(DD1-PadL16)
- DD1 pad R19: (no net) -> GNDD
- DD1 pad R22: (no net) -> Net-(DD1-PadL16)
- DD1 pad R23: (no net) -> GNDD
- DD1 pad R8: (no net) -> Net-(DD1-PadL16)
- DD1 pad R9: (no net) -> Net-(DD1-PadL16)
- DD1 pad T10: (no net) -> GNDD
- DD1 pad T11: (no net) -> GNDD
- DD1 pad T12: (no net) -> GNDD
- DD1 pad T13: (no net) -> GNDD
- DD1 pad T14: (no net) -> GNDD
- DD1 pad T15: (no net) -> GNDD
- DD1 pad T16: (no net) -> GNDD
- DD1 pad T8: (no net) -> GNDD
- DD1 pad T9: (no net) -> GNDD
- DD1 pad U10: (no net) -> Net-(DD1-PadL16)
- DD1 pad U11: (no net) -> Net-(DD1-PadL16)
- DD1 pad U12: (no net) -> Net-(DD1-PadL16)
- DD1 pad U13: (no net) -> Net-(DD1-PadL16)
- DD1 pad U14: (no net) -> Net-(DD1-PadL16)
- DD1 pad U15: (no net) -> Net-(DD1-PadL16)
- DD1 pad U16: (no net) -> Net-(DD1-PadL16)
- DD1 pad U19: (no net) -> GNDD
- DD1 pad U2: (no net) -> GNDD
- DD1 pad U22: (no net) -> GNDD
- DD1 pad U8: (no net) -> Net-(DD1-PadL16)
- DD1 pad U9: (no net) -> Net-(DD1-PadL16)
- DD1 pad V10: (no net) -> GNDD
- DD1 pad V11: (no net) -> GNDD
- DD1 pad V12: (no net) -> GNDD
- DD1 pad V13: (no net) -> GNDD
- DD1 pad V14: (no net) -> GNDD
- DD1 pad V15: (no net) -> GNDD
- DD1 pad V16: (no net) -> GNDD
- DD1 pad V3: (no net) -> Net-(DD1-PadL16)
- DD1 pad V8: (no net) -> GNDD
- DD1 pad V9: (no net) -> GNDD
- DD1 pad W14: (no net) -> GNDD
- DD1 pad W20: (no net) -> GNDD
- DD1 pad W22: (no net) -> Net-(DD1-PadL16)
- DD1 pad W23: (no net) -> GNDD
- DD1 pad W9: (no net) -> GNDD
- DD1 pad Y11: (no net) -> GNDD
- DD1 pad Y19: (no net) -> GNDD
- J1 pad 137: (no net) -> GNDD
- J1 pad 138: (no net) -> GNDD
- J1 pad 14: (no net) -> GNDD
- J1 pad 143: (no net) -> GNDD
- J1 pad 146: (no net) -> GNDD
- J1 pad 149: (no net) -> GNDD
- J1 pad 152: (no net) -> GNDD
- J1 pad 155: (no net) -> GNDD
- J1 pad 158: (no net) -> GNDD
- J1 pad 163: (no net) -> GNDD
- J1 pad 164: (no net) -> GNDD
- J1 pad 169: (no net) -> GNDD
- J1 pad 17: (no net) -> GNDD
- J1 pad 170: (no net) -> GNDD
- J1 pad 175: (no net) -> GNDD
- J1 pad 178: (no net) -> GNDD
- J1 pad 181: (no net) -> GNDD
- J1 pad 184: (no net) -> GNDD
- J1 pad 187: (no net) -> GNDD
- J1 pad 190: (no net) -> GNDD
- J1 pad 195: (no net) -> GNDD
- J1 pad 196: (no net) -> GNDD
- J1 pad 2: (no net) -> GNDD
- J1 pad 20: (no net) -> GNDD
- J1 pad 23: (no net) -> GNDD
- J1 pad 26: (no net) -> GNDD
- J1 pad 29: (no net) -> GNDD
- J1 pad 3: (no net) -> GNDD
- J1 pad 32: (no net) -> GNDD
- J1 pad 35: (no net) -> GNDD
- J1 pad 38: (no net) -> GNDD
- J1 pad 41: (no net) -> GNDD
- J1 pad 46: (no net) -> GNDD
- J1 pad 47: (no net) -> GNDD
- J1 pad 52: (no net) -> GNDD
- J1 pad 53: (no net) -> GNDD
- J1 pad 58: (no net) -> GNDD
- J1 pad 61: (no net) -> GNDD
- J1 pad 64: (no net) -> GNDD
- J1 pad 67: (no net) -> GNDD
- J1 pad 70: (no net) -> GNDD
- J1 pad 73: (no net) -> GNDD
- J1 pad 78: (no net) -> GNDD
- J1 pad 79: (no net) -> GNDD
- J1 pad 8: (no net) -> GNDD
- J1 pad 9: (no net) -> GNDD

Commit message: Work in progress...
Connections:
- J1 pad 101: (no net) -> +1V35
- J1 pad 102: (no net) -> +1V35
- J1 pad 109: (no net) -> +1V35
- J1 pad 110: (no net) -> +1V35
- J1 pad 115: (no net) -> +1V35
- J1 pad 116: (no net) -> +1V35
- J1 pad 123: (no net) -> +1V35
- J1 pad 124: (no net) -> +1V35
- J1 pad 131: (no net) -> +1V35
- J1 pad 132: (no net) -> +1V35
- J1 pad 85: (no net) -> +1V35
- J1 pad 86: (no net) -> +1V35
- J1 pad 93: (no net) -> +1V35
- J1 pad 94: (no net) -> +1V35
Changed lines of the file:
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@@
     (zones 0)
     (modules 2)
-    (nets 5)
+    (nets 6)
   )
   (page A4 portrait)
@@
   (net 3 "Net-(DD1-PadL16)")
   (net 4 "Net-(DD1-PadA1)")
+  (net 5 +1V35)
   (net_class Default "Это класс цепей по умолчанию."
     (clearance 0.2)
@@
     (uvia_dia 0.3)
     (uvia_drill 0.1)
+    (add_net +1V35)
     (add_net GNDD)
     (add_net "Net-(DD1-PadA1)")
@@
     (pad 81 smd rect (at -4.1 5.25) (size 2 0.35) (layers B.Cu B.Paste B.Mask))
     (pad 83 smd rect (at -4.1 4.65) (size 2 0.35) (layers B.Cu B.Paste B.Mask))
-    (pad 85 smd rect (at -4.1 4.05) (size 2 0.35) (layers B.Cu B.Paste B.Mask))
+    (pad 85 smd rect (at -4.1 4.05) (size 2 0.35) (layers B.Cu B.Paste B.Mask)
+      (net 5 +1V35))
     (pad 87 smd rect (at -4.1 3.45) (size 2 0.35) (layers B.Cu B.Paste B.Mask))
     (pad 89 smd rect (at -4.1 2.85) (size 2 0.35) (layers B.Cu B.Paste B.Mask))
     (pad 91 smd rect (at -4.1 2.25) (size 2 0.35) (layers B.Cu B.Paste B.Mask))
-    (pad 93 smd rect (at -4.1 1.65) (size 2 0.35) (layers B.Cu B.Paste B.Mask))
+    (pad 93 smd rect (at -4.1 1.65) (size 2 0.35) (layers B.Cu B.Paste B.Mask)
+      (net 5 +1V35))
     (pad 95 smd rect (at -4.1 1.05) (size 2 0.35) (layers B.Cu B.Paste B.Mask))
     (pad 97 smd rect (at -4.1 0.45) (size 2 0.35) (layers B.Cu B.Paste B.Mask))
     (pad 99 smd rect (at -4.1 -0.15) (size 2 0.35) (layers B.Cu B.Paste B.Mask))
-    (pad 101 smd rect (at -4.1 -0.75) (size 2 0.35) (layers B.Cu B.Paste B.Mask))
+    (pad 101 smd rect (at -4.1 -0.75) (size 2 0.35) (layers B.Cu B.Paste B.Mask)
+      (net 5 +1V35))
     (pad 103 smd rect (at -4.1 -1.35) (size 2 0.35) (layers B.Cu B.Paste B.Mask))
     (pad 105 smd rect (at -4.1 -1.95) (size 2 0.35) (layers B.Cu B.Paste B.Mask))
     (pad 107 smd rect (at -4.1 -2.55) (size 2 0.35) (layers B.Cu B.Paste B.Mask))
-    (pad 109 smd rect (at -4.1 -3.15) (size 2 0.35) (layers B.Cu B.Paste B.Mask))
+    (pad 109 smd rect (at -4.1 -3.15) (size 2 0.35) (layers B.Cu B.Paste B.Mask)
+      (net 5 +1V35))
     (pad 111 smd rect (at -4.1 -3.75) (size 2 0.35) (layers B.Cu B.Paste B.Mask))
     (pad 113 smd rect (at -4.1 -4.35) (size 2 0.35) (layers B.Cu B.Paste B.Mask))
-    (pad 115 smd rect (at -4.1 -4.95) (size 2 0.35) (layers B.Cu B.Paste B.Mask))
+    (pad 115 smd rect (at -4.1 -4.95) (size 2 0.35) (layers B.Cu B.Paste B.Mask)
+      (net 5 +1V35))
     (pad 117 smd rect (at -4.1 -5.55) (size 2 0.35) (layers B.Cu B.Paste B.Mask))
     (pad 119 smd rect (at -4.1 -6.15) (size 2 0.35) (layers B.Cu B.Paste B.Mask))
     (pad 121 smd rect (at -4.1 -6.75) (size 2 0.35) (layers B.Cu B.Paste B.Mask))
-    (pad 123 smd rect (at -4.1 -7.35) (size 2 0.35) (layers B.Cu B.Paste B.Mask))
+    (pad 123 smd rect (at -4.1 -7.35) (size 2 0.35) (layers B.Cu B.Paste B.Mask)
+      (net 5 +1V35))
     (pad 125 smd rect (at -4.1 -7.95) (size 2 0.35) (layers B.Cu B.Paste B.Mask))
     (pad 127 smd rect (at -4.1 -8.55) (size 2 0.35) (layers B.Cu B.Paste B.Mask))
     (pad 129 smd rect (at -4.1 -9.15) (size 2 0.35) (layers B.Cu B.Paste B.Mask))
-    (pad 131 smd rect (at -4.1 -9.75) (size 2 0.35) (layers B.Cu B.Paste B.Mask))
+    (pad 131 smd rect (at -4.1 -9.75) (size 2 0.35) (layers B.Cu B.Paste B.Mask)
+      (net 5 +1V35))
     (pad 133 smd rect (at -4.1 -10.35) (size 2 0.35) (layers B.Cu B.Paste B.Mask))
     (pad 135 smd rect (at -4.1 -10.95) (size 2 0.35) (layers B.Cu B.Paste B.Mask))
@@
     (pad 82 smd rect (at 4.1 4.95) (size 2 0.35) (layers B.Cu B.Paste B.Mask))
     (pad 84 smd rect (at 4.1 4.35) (size 2 0.35) (layers B.Cu B.Paste B.Mask))
-    (pad 86 smd rect (at 4.1 3.75) (size 2 0.35) (layers B.Cu B.Paste B.Mask))
+    (pad 86 smd rect (at 4.1 3.75) (size 2 0.35) (layers B.Cu B.Paste B.Mask)
+      (net 5 +1V35))
     (pad 88 smd rect (at 4.1 3.15) (size 2 0.35) (layers B.Cu B.Paste B.Mask))
     (pad 90 smd rect (at 4.1 2.55) (size 2 0.35) (layers B.Cu B.Paste B.Mask))
     (pad 92 smd rect (at 4.1 1.95) (size 2 0.35) (layers B.Cu B.Paste B.Mask))
-    (pad 94 smd rect (at 4.1 1.35) (size 2 0.35) (layers B.Cu B.Paste B.Mask))
+    (pad 94 smd rect (at 4.1 1.35) (size 2 0.35) (layers B.Cu B.Paste B.Mask)
+      (net 5 +1V35))
     (pad 96 smd rect (at 4.1 0.75) (size 2 0.35) (layers B.Cu B.Paste B.Mask))
     (pad 98 smd rect (at 4.1 0.15) (size 2 0.35) (layers B.Cu B.Paste B.Mask))
     (pad 100 smd rect (at 4.1 -0.45) (size 2 0.35) (layers B.Cu B.Paste B.Mask))
-    (pad 102 smd rect (at 4.1 -1.05) (size 2 0.35) (layers B.Cu B.Paste B.Mask))
+    (pad 102 smd rect (at 4.1 -1.05) (size 2 0.35) (layers B.Cu B.Paste B.Mask)
+      (net 5 +1V35))
     (pad 104 smd rect (at 4.1 -1.65) (size 2 0.35) (layers B.Cu B.Paste B.Mask))
     (pad 106 smd rect (at 4.1 -2.25) (size 2 0.35) (layers B.Cu B.Paste B.Mask))
     (pad 108 smd rect (at 4.1 -2.85) (size 2 0.35) (layers B.Cu B.Paste B.Mask))
-    (pad 110 smd rect (at 4.1 -3.45) (size 2 0.35) (layers B.Cu B.Paste B.Mask))
+    (pad 110 smd rect (at 4.1 -3.45) (size 2 0.35) (layers B.Cu B.Paste B.Mask)
+      (net 5 +1V35))
     (pad 112 smd rect (at 4.1 -4.05) (size 2 0.35) (layers B.Cu B.Paste B.Mask))
     (pad 114 smd rect (at 4.1 -4.65) (size 2 0.35) (layers B.Cu B.Paste B.Mask))
-    (pad 116 smd rect (at 4.1 -5.25) (size 2 0.35) (layers B.Cu B.Paste B.Mask))
+    (pad 116 smd rect (at 4.1 -5.25) (size 2 0.35) (layers B.Cu B.Paste B.Mask)
+      (net 5 +1V35))
     (pad 118 smd rect (at 4.1 -5.85) (size 2 0.35) (layers B.Cu B.Paste B.Mask))
     (pad 120 smd rect (at 4.1 -6.45) (size 2 0.35) (layers B.Cu B.Paste B.Mask))
     (pad 122 smd rect (at 4.1 -7.05) (size 2 0.35) (layers B.Cu B.Paste B.Mask))
-    (pad 124 smd rect (at 4.1 -7.65) (size 2 0.35) (layers B.Cu B.Paste B.Mask))
+    (pad 124 smd rect (at 4.1 -7.65) (size 2 0.35) (layers B.Cu B.Paste B.Mask)
+      (net 5 +1V35))
     (pad 126 smd rect (at 4.1 -8.25) (size 2 0.35) (layers B.Cu B.Paste B.Mask))
     (pad 128 smd rect (at 4.1 -8.85) (size 2 0.35) (layers B.Cu B.Paste B.Mask))
     (pad 130 smd rect (at 4.1 -9.45) (size 2 0.35) (layers B.Cu B.Paste B.Mask))
-    (pad 132 smd rect (at 4.1 -10.05) (size 2 0.35) (layers B.Cu B.Paste B.Mask))
+    (pad 132 smd rect (at 4.1 -10.05) (size 2 0.35) (layers B.Cu B.Paste B.Mask)
+      (net 5 +1V35))
     (pad 134 smd rect (at 4.1 -10.65) (size 2 0.35) (layers B.Cu B.Paste B.Mask))
     (pad 136 smd rect (at 4.1 -11.25) (size 2 0.35) (layers B.Cu B.Paste B.Mask))

Commit message: Added new schematic sheets.
Connections:
- DD1 pad A24: (no net) -> +1V5
- DD1 pad AA19: (no net) -> /CPU/DDR3/DQ0
- DD1 pad AA22: (no net) -> /CPU/DDR3/DQ1
- DD1 pad AB22: (no net) -> +1V5
- DD1 pad AB23: (no net) -> /CPU/DDR3/DQ2
- DD1 pad AB24: (no net) -> /CPU/DDR3/DQ3
- DD1 pad AB3: (no net) -> Net-(DD1-PadAB3)
- DD1 pad AC22: (no net) -> /CPU/DDR3/DM0
- DD1 pad AD24: (no net) -> +1V5
- DD1 pad C10: (no net) -> Net-(DD1-PadAB3)
- DD1 pad C12: (no net) -> Net-(DD1-PadAB3)
- DD1 pad C22: (no net) -> +1V5
- DD1 pad C4: (no net) -> Net-(DD1-PadAB3)
- DD1 pad C6: (no net) -> Net-(DD1-PadAB3)
- DD1 pad C7: (no net) -> Net-(DD1-PadAB3)
- DD1 pad D20: (no net) -> +1V5
- DD1 pad F19: (no net) -> +1V5
- DD1 pad F3: (no net) -> Net-(DD1-PadAB3)
- DD1 pad G24: (no net) -> +1V5
- DD1 pad H19: (no net) -> +1V5
- DD1 pad H3: (no net) -> Net-(DD1-PadAB3)
- DD1 pad J24: (no net) -> +1V5
- DD1 pad K21: (no net) -> +1V5
- DD1 pad L19: (no net) -> +1V5
- DD1 pad L24: (no net) -> +1V5
- DD1 pad L3: (no net) -> Net-(DD1-PadAB3)
- DD1 pad N18: (no net) -> +1V5
- DD1 pad N21: (no net) -> +1V5
- DD1 pad N24: (no net) -> +1V5
- DD1 pad P23: (no net) -> /CPU/DDR3/DQ17
- DD1 pad P24: (no net) -> /CPU/DDR3/DQ18
- DD1 pad P3: (no net) -> Net-(DD1-PadAB3)
- DD1 pad R20: (no net) -> +1V5
- DD1 pad R21: (no net) -> /CPU/DDR3/DQ19
- DD1 pad R24: (no net) -> +1V5
- DD1 pad T23: (no net) -> /CPU/DDR3/DQS2
- DD1 pad T24: (no net) -> /CPU/DDR3/DQS_N2
- DD1 pad T3: (no net) -> Net-(DD1-PadAB3)
- DD1 pad U20: (no net) -> +1V5
- DD1 pad U23: (no net) -> +1V5
- DD1 pad V20: (no net) -> /CPU/DDR3/DQ16
- DD1 pad V22: (no net) -> /CPU/DDR3/DQ8
- DD1 pad V23: (no net) -> /CPU/DDR3/DQ9
- DD1 pad V24: (no net) -> /CPU/DDR3/DQ10
- DD1 pad W24: (no net) -> +1V5
- DD1 pad W3: (no net) -> Net-(DD1-PadAB3)
- DD1 pad Y17: (no net) -> Net-(DD1-PadAB3)
- DD1 pad Y20: (no net) -> +1V5
- DD1 pad Y22: (no net) -> /CPU/DDR3/DQ11
- DD1 pad Y23: (no net) -> /CPU/DDR3/DQS1
- DD1 pad Y24: (no net) -> /CPU/DDR3/DQS_N1
- J1 pad 11: (no net) -> /CPU/DDR3/DM0
- J1 pad 13: (no net) -> /CPU/DDR3/DQ2
- J1 pad 15: (no net) -> /CPU/DDR3/DQ3
- J1 pad 19: (no net) -> /CPU/DDR3/DQ8
- J1 pad 21: (no net) -> /CPU/DDR3/DQ9
- J1 pad 25: (no net) -> /CPU/DDR3/DQS_N1
- J1 pad 27: (no net) -> /CPU/DDR3/DQS1
- J1 pad 31: (no net) -> /CPU/DDR3/DQ10
- J1 pad 33: (no net) -> /CPU/DDR3/DQ11
- J1 pad 37: (no net) -> /CPU/DDR3/DQ16
- J1 pad 39: (no net) -> /CPU/DDR3/DQ17
- J1 pad 43: (no net) -> /CPU/DDR3/DQS_N2
- J1 pad 45: (no net) -> /CPU/DDR3/DQS2
- J1 pad 49: (no net) -> /CPU/DDR3/DQ18
- J1 pad 5: (no net) -> /CPU/DDR3/DQ0
- J1 pad 51: (no net) -> /CPU/DDR3/DQ19
- J1 pad 7: (no net) -> /CPU/DDR3/DQ1
Other:
- copper layers 2 -> 4
